File: PD_PowerSupply.sch (KiCad schematic (older format))
At the start: 29 parts, among them J1 USB4085-GF-A_REVA, Q1 STL6P3LLH6, Q2 STL6P3LLH6, U1 STUSB4500QTR, U2 ESP32-WROOM-32, U3 CP2102N, U4 IR38062MTRPBF, U5 IR38062MTRPBF

Commit message: switched to linear chip
Parts:
- removed U4, U5: IR38062MTRPBF, PQFN50P700X500X100-26N, symbol IR38062MTRPBF:IR38062MTRPBF
- added U6: LTC3886, Package_DFN_QFN:Linear_UGK52_QFN-46-52, symbol Regulator_Switching:LTC3886
Connections:
- wire segments 111 -> 121
- no-connect marks 5 -> 11
Other:
- note added: "Might switch to NRF52 due to PMBus compatibility issues \n"
- moved on the sheet: R10, R9, U2, U3
Changed lines of the file:
@@
 L RF_Module:ESP32-WROOM-32 U2
 U 1 1 5E77E77E
-P 1500 6500
-F 0 "U2" H 1050 7850 50  0000 C CNN
-F 1 "ESP32-WROOM-32" V 950 5550 50  0000 C CNN
-F 2 "RF_Module:ESP32-WROOM-32" H 1500 5000 50  0001 C CNN
-F 3 "https://www.espressif.com/sites/default/files/documentation/esp32-wroom-32_datasheet_en.pdf" H 1200 6550 50  0001 C CNN
-	1    1500 6500
-	1    0    0    -1
-$EndComp
-Text Label 3350 6700 0    50   ~ 0
+P 1950 6150
+F 0 "U2" H 1500 7500 50  0000 C CNN
+F 1 "ESP32-WROOM-32" V 1400 5200 50  0000 C CNN
+F 2 "RF_Module:ESP32-WROOM-32" H 1950 4650 50  0001 C CNN
+F 3 "https://www.espressif.com/sites/default/files/documentation/esp32-wroom-32_datasheet_en.pdf" H 1650 6200 50  0001 C CNN
+	1    1950 6150
+	1    0    0    -1
+$EndComp
+Text Label 3800 6350 0    50   ~ 0
 I2C_SDA
-Text Label 3350 6800 0    50   ~ 0
+Text Label 3800 6450 0    50   ~ 0
 I2C_SCL
-Text Notes 3800 6800 0    50   ~ 0
+Text Notes 4250 6450 0    50   ~ 0
 add test header
 Wire Wire Line
-	2100 6700 2750 6700
-Wire Wire Line
-	2100 6800 3050 6800
+	2550 6350 3200 6350
+Wire Wire Line
+	2550 6450 3500 6450
 $Comp
 L Device:R_US R9
 U 1 1 5E787840
-P 2750 6500
-F 0 "R9" H 2818 6546 50  0000 L CNN
-F 1 "4.7k" H 2818 6455 50  0000 L CNN
-F 2 "" V 2790 6490 50  0001 C CNN
-F 3 "~" H 2750 6500 50  0001 C CNN
-	1    2750 6500
+P 3200 6150
+F 0 "R9" H 3268 6196 50  0000 L CNN
+F 1 "4.7k" H 3268 6105 50  0000 L CNN
+F 2 "" V 3240 6140 50  0001 C CNN
+F 3 "~" H 3200 6150 50  0001 C CNN
+	1    3200 6150
 	1    0    0    -1
 $EndComp
@@
 L Device:R_US R10
 U 1 1 5E788698
-P 3050 6500
-F 0 "R10" H 3118 6546 50  0000 L CNN
-F 1 "4.7k" H 3118 6455 50  0000 L CNN
-F 2 "" V 3090 6490 50  0001 C CNN
-F 3 "~" H 3050 6500 50  0001 C CNN
-	1    3050 6500
-	1    0    0    -1
-$EndComp
-Wire Wire Line
-	2750 6650 2750 6700
-Connection ~ 2750 6700
-Wire Wire Line
-	2750 6700 3350 6700
-Wire Wire Line
-	3050 6650 3050 6800
-Connection ~ 3050 6800
-Wire Wire Line
-	3050 6800 3350 6800
+P 3500 6150
+F 0 "R10" H 3568 6196 50  0000 L CNN
+F 1 "4.7k" H 3568 6105 50  0000 L CNN
+F 2 "" V 3540 6140 50  0001 C CNN
+F 3 "~" H 3500 6150 50  0001 C CNN
+	1    3500 6150
+	1    0    0    -1
+$EndComp
+Wire Wire Line
+	3200 6300 3200 6350
+Connection ~ 3200 6350
+Wire Wire Line
+	3200 6350 3800 6350
+Wire Wire Line
+	3500 6300 3500 6450
+Connection ~ 3500 6450
+Wire Wire Line
+	3500 6450 3800 6450
 $Comp
 L power:+2V7 #PWR0101
 U 1 1 5E78B272
-P 2750 6350
-F 0 "#PWR0101" H 2750 6200 50  0001 C CNN
-F 1 "+2V7" H 2765 6523 50  0000 C CNN
-F 2 "" H 2750 6350 50  0001 C CNN
-F 3 "" H 2750 6350 50  0001 C CNN
-	1    2750 6350
+P 3200 6000
+F 0 "#PWR0101" H 3200 5850 50  0001 C CNN
+F 1 "+2V7" H 3215 6173 50  0000 C CNN
+F 2 "" H 3200 6000 50  0001 C CNN
+F 3 "" H 3200 6000 50  0001 C CNN
+	1    3200 6000
 	1    0    0    -1
 $EndComp
@@
 L power:+2V7 #PWR0102
 U 1 1 5E78BB5A
-P 3050 6350
-F 0 "#PWR0102" H 3050 6200 50  0001 C CNN
-F 1 "+2V7" H 3065 6523 50  0000 C CNN
-F 2 "" H 3050 6350 50  0001 C CNN
-F 3 "" H 3050 6350 50  0001 C CNN
-	1    3050 6350
+P 3500 6000
+F 0 "#PWR0102" H 3500 5850 50  0001 C CNN
+F 1 "+2V7" H 3515 6173 50  0000 C CNN
+F 2 "" H 3500 6000 50  0001 C CNN
+F 3 "" H 3500 6000 50  0001 C CNN
+	1    3500 6000
 	1    0    0    -1
 $EndComp
@@
 Text Label 3800 3000 0    50   ~ 0
 STUSB_ALERT
-Text Label 2400 7600 0    50   ~ 0
+Text Label 2850 7250 0    50   ~ 0
 STUSB_ALERT
 Wire Wire Line
-	2400 7600 2100 7600
+	2850 7250 2550 7250
 $Comp
 L Device:D_Schottky D1
@@
 Text Label 3800 2200 0    50   ~ 0
 STUSB_RESET
-Text Label 2400 7500 0    50   ~ 0
+Text Label 2850 7150 0    50   ~ 0
 STUSB_RESET
 Wire Wire Line
-	2400 7500 2100 7500
+	2850 7150 2550 7150
 Wire Wire Line
 	3550 2250 3550 2200
@@
 L Interface_USB:CP2102N-A01-GQFN24 U3
 U 1 1 5E78F2C6
-P 6450 6950
-F 0 "U3" H 6050 7750 50  0000 C CNN
-F 1 "CP2102N" H 6750 7750 50  0000 C CNN
-F 2 "Package_DFN_QFN:QFN-24-1EP_4x4mm_P0.5mm_EP2.6x2.6mm" H 6900 6150 50  0001 L CNN
-F 3 "https://www.silabs.com/documents/public/data-sheets/cp2102n-datasheet.pdf" H 6500 5900 50  0001 C CNN
-	1    6450 6950
-	1    0    0    -1
-$EndComp
-Text Label 5350 7350 0    50   ~ 0
+P 2000 9250
+F 0 "U3" H 1600 10050 50  0000 C CNN
+F 1 "CP2102N" H 2300 10050 50  0000 C CNN
+F 2 "Package_DFN_QFN:QFN-24-1EP_4x4mm_P0.5mm_EP2.6x2.6mm" H 2450 8450 50  0001 L CNN
+F 3 "https://www.silabs.com/documents/public/data-sheets/cp2102n-datasheet.pdf" H 2050 8200 50  0001 C CNN
+	1    2000 9250
+	1    0    0    -1
+$EndComp
+Text Label 900  9650 0    50   ~ 0
 USB_DP
-Text Label 5350 7450 0    50   ~ 0
+Text Label 900  9750 0    50   ~ 0
 USB_DN
 Wire Wire Line
-	5350 7450 5850 7450
-Wire Wire Line
-	5350 7350 5850 7350
+	900  9750 1400 9750
+Wire Wire Line
+	900  9650 1400 9650
 $Comp
 L power:GND #PWR0112
 U 1 1 5E7978C1
-P 6500 7950
-F 0 "#PWR0112" H 6500 7700 50  0001 C CNN
-F 1 "GND" H 6505 7777 50  0000 C CNN
-F 2 "" H 6500 7950 50  0001 C CNN
-F 3 "" H 6500 7950 50  0001 C CNN
-	1    6500 7950
-	1    0    0    -1
-$EndComp
-Wire Wire Line
-	6500 7950 6500 7850
-Wire Wire Line
-	6500 7850 6550 7850
-Wire Wire Line
-	6450 7850 6500 7850
-Connection ~ 6500 7850
+P 2050 10250
+F 0 "#PWR0112" H 2050 10000 50  0001 C CNN
+F 1 "GND" H 2055 10077 50  0000 C CNN
+F 2 "" H 2050 10250 50  0001 C CNN
+F 3 "" H 2050 10250 50  0001 C CNN
+	1    2050 10250
+	1    0    0    -1
+$EndComp
+Wire Wire Line
+	2050 10250 2050 10150
+Wire Wire Line
+	2050 10150 2100 10150
+Wire Wire Line
+	2000 10150 2050 10150
+Connection ~ 2050 10150
 $Comp
 L power:+3.3V #PWR0113
 U 1 1 5E782AC4
-P 1500 5050
-F 0 "#PWR0113" H 1500 4900 50  0001 C CNN
-F 1 "+3.3V" H 1515 5223 50  0000 C CNN
-F 2 "" H 1500 5050 50  0001 C CNN
-F 3 "" H 1500 5050 50  0001 C CNN
-	1    1500 5050
-	1    0    0    -1
-$EndComp
-Wire Wire Line
-	1500 5050 1500 5100
+P 1950 4700
+F 0 "#PWR0113" H 1950 4550 50  0001 C CNN
+F 1 "+3.3V" H 1965 4873 50  0000 C CNN
+F 2 "" H 1950 4700 50  0001 C CNN
+F 3 "" H 1950 4700 50  0001 C CNN
+	1    1950 4700
+	1    0    0    -1
+$EndComp
+Wire Wire Line
+	1950 4700 1950 4750
 Text Label 8450 1000 0    50   ~ 0
 vSINK
 $Comp
-L power:VBUS #PWR?
+L power:VBUS #PWR0114
 U 1 1 5E78E73B
 P 1900 950
-F 0 "#PWR?" H 1900 800 50  0001 C CNN
+F 0 "#PWR0114" H 1900 800 50  0001 C CNN
 F 1 "VBUS" H 1900 1150 50  0000 C CNN
 F 2 "" H 1900 950 50  0001 C CNN
@@
 Wire Wire Line
 	1900 1000 2700 1000
-$Comp
-L IR38062MTRPBF:IR38062MTRPBF U4
-U 1 1 5E7944E7
-P 11100 2950
-F 0 "U4" H 11100 4417 50  0000 C CNN
-F 1 "IR38062MTRPBF" H 11100 4326 50  0000 C CNN
-F 2 "PQFN50P700X500X100-26N" H 11100 2950 50  0001 L BNN
-F 3 "Infineon" H 11100 2950 50  0001 L BNN
-	1    11100 2950
-	1    0    0    -1
-$EndComp
-$Comp
-L IR38062MTRPBF:IR38062MTRPBF U5
-U 1 1 5E797DCB
-P 11100 6950
-F 0 "U5" H 11100 8417 50  0000 C CNN
-F 1 "IR38062MTRPBF" H 11100 8326 50  0000 C CNN
-F 2 "PQFN50P700X500X100-26N" H 11100 6950 50  0001 L BNN
-F 3 "Infineon" H 11100 6950 50  0001 L BNN
-	1    11100 6950
-	1    0    0    -1
-$EndComp
+NoConn ~ 1450 2550
+NoConn ~ 1450 2650
+$Comp
+L Regulator_Switching:LTC3886 U6
+U 1 1 5E795D79
+P 10900 3900
+F 0 "U6" H 11450 4050 50  0000 C CNN
+F 1 "LTC3886" H 10450 4050 50  0000 C CNN
+F 2 "Package_DFN_QFN:Linear_UGK52_QFN-46-52" H 11200 750 50  0001 L CNN
+F 3 "https://www.analog.com/media/en/technical-documentation/data-sheets/LTC3886-3886-1.pdf" H 10900 4250 50  0001 C CNN
+	1    10900 3900
+	1    0    0    -1
+$EndComp
+$Comp
+L power:GND #PWR?
+U 1 1 5E7B1077
+P 1950 7600
+F 0 "#PWR?" H 1950 7350 50  0001 C CNN
+F 1 "GND" H 1955 7427 50  0000 C CNN
+F 2 "" H 1950 7600 50  0001 C CNN
+F 3 "" H 1950 7600 50  0001 C CNN
+	1    1950 7600
+	1    0    0    -1
+$EndComp
+Wire Wire Line
+	1950 7600 1950 7550
+$Comp
+L power:+3.3V #PWR?
+U 1 1 5E7B5A1B
+P 1950 8300
+F 0 "#PWR?" H 1950 8150 50  0001 C CNN
+F 1 "+3.3V" H 1965 8473 50  0000 C CNN
+F 2 "" H 1950 8300 50  0001 C CNN
+F 3 "" H 1950 8300 50  0001 C CNN
+	1    1950 8300
+	1    0    0    -1
+$EndComp
+Wire Wire Line
+	1950 8300 1950 8350
+Wire Wire Line
+	1950 8350 1900 8350
+Wire Wire Line
+	1950 8350 2000 8350
+Connection ~ 1950 8350
+Wire Wire Line
+	2600 8950 2700 8950
+Wire Wire Line
+	2700 8950 2700 5050
+Wire Wire Line
+	2700 5050 2550 5050
+Wire Wire Line
+	2600 9050 2750 9050
+Wire Wire Line
+	2750 9050 2750 5250
+Wire Wire Line
+	2750 5250 2550 5250
+NoConn ~ 2600 9850
+NoConn ~ 2600 9750
+NoConn ~ 2600 9650
+NoConn ~ 2600 9550
+Text Notes 2850 5350 0    50   ~ 0
+Might switch to NRF52 due to PMBus compatibility issues \n
 $EndSCHEMATC

Commit message: switched to unswitched
Parts:
- added C? (x16): C, symbol Device:C
- added L? (x2): L, symbol Device:L
- added R? (x10): R_US, symbol Device:R_US
- added U4, U5: IR38062MTRPBF, PQFN50P700X500X100-26N, symbol IR38062MTRPBF:IR38062MTRPBF
Connections:
- net labels added: PGOOD_CH0, PGOOD_CH1, VOUT_CH0, VOUT_CH1
- wire segments 121 -> 246

Commit message: added footprints and symbol for LTC2972
Parts:
- removed C? (x16): C, symbol Device:C
- removed L? (x2): L, symbol Device:L
- removed R? (x10): R_US, symbol Device:R_US
- removed U4, U5: IR38062MTRPBF, PQFN50P700X500X100-26N, symbol IR38062MTRPBF:IR38062MTRPBF
- removed U6: LTC3886, Package_DFN_QFN:Linear_UGK52_QFN-46-52, symbol Regulator_Switching:LTC3886
- added U4, U5: LTM8074IY#PBF, BGA25C65P5X5_400X400X198N, symbol LTM8074IY_PBF:LTM8074IY#PBF
- added U?: LTC2972, LTC2972:LTC2972, symbol LTC2972_SCH:LTC2972
Connections:
- net labels removed: PGOOD_CH0, PGOOD_CH1, VOUT_CH0, VOUT_CH1
- wire segments 246 -> 123

Commit message: set up coprocessor
Parts:
- removed R10: 4.7k, symbol Device:R_US
- removed U2: ESP32-WROOM-32, RF_Module:ESP32-WROOM-32, symbol RF_Module:ESP32-WROOM-32
- removed U3: CP2102N, Package_DFN_QFN:QFN-24-1EP_4x4mm_P0.5mm_EP2.6x2.6mm, symbol Interface_USB:CP2102N-A01-GQFN24
- added C10, C11: C, symbol Device:C
- added C12, C13: 10nF, symbol Device:C
- added C6: .01uF, symbol Device:C
- added C7, C8, C9, C? (x3): .1uF, symbol Device:C
- added DBG1: Cortex Debug, symbol Connector:Conn_ARM_JTAG_SWD_10
- added J1, J2: Connector, symbol Connector:Conn_01x02_Male
- added Q3, Q4: MMBT3906, Package_TO_SOT_SMD:SOT-23, symbol Transistor_BJT:MMBT3906
- added R12, R17, R20, R24: R_US, symbol Device:R_US
- added R13, R15, R23: R_Shunt_US, symbol Device:R_Shunt_US
- added R14, R16, R18, R19, R21, R22: 10k, symbol Device:R_US
- added R? (x4): 47.5k, symbol Device:R_US
- added U2: nRF52840, Package_DFN_QFN:Nordic_AQFN-73-1EP_7x7mm_P0.5mm, symbol MCU_Nordic:nRF52840
- added U3: STM32L432KCUx, Package_DFN_QFN:QFN-32-1EP_5x5mm_P0.5mm_EP3.45x3.45mm, symbol MCU_ST_STM32L4:STM32L432KCUx
- R9: value 4.7k -> 10k
- gave numbers to parts that had none: 1
- renumbered J1 to USB1
Connections:
- net +2V8 is gone; now on net +3V3: R9.1
- net +3V3: now also U6.25 (VDDIO), C?.1, C?.1, C?.1, DBG1.1 (VTref), R14.1, R16.1, R18.1, R19.1, R21.1, R22.1, R?.1, R?.1, R?.1, R?.1, U2.A22 (VDD), U2.AD14 (VDD), U2.AD2 (VBUS), U2.AD23 (VDD), U2.B1 (VDD), U2.W1 (VDD), U2.Y2 (VDDH), U3.1 (VDD), U3.17 (VDD), U3.5 (VDDA)
- net GND: now also U4.A1 (GND), U4.A5 (GND), U4.B2 (GND), U4.B3 (GND), U4.B4 (GND), U4.C2 (GND), U4.C3 (GND), U4.C4 (GND), U4.C5 (GND), U4.D2 (GND), U4.D3 (GND), U4.D4 (GND), U4.E3 (GND), U4.E4 (GND), U4.E5 (GND), U5.A1 (GND), U5.A5 (GND), U5.B2 (GND), U5.B3 (GND), U5.B4 (GND), U5.C2 (GND), U5.C3 (GND), U5.C4 (GND), U5.C5 (GND), U5.D2 (GND), U5.D3 (GND), U5.D4 (GND), U5.E3 (GND), U5.E4 (GND), U5.E5 (GND), U6.19 (WP), U6.26 (ASEL0), U6.27 (ASEL1), U6.33 (VSENSEM0), U6.37 (VSENSEM1), C10.1, C11.1, C12.1, C13.1, C6.2, C8.1, C9.1, C?.2, C?.2, C?.2, DBG1.3 (GND), DBG1.5 (GND), DBG1.9 (GNDDetect), J1.2 (Pin_2), J2.2 (Pin_2), Q3.1 (B), Q3.3 (C), Q4.1 (B), Q4.3 (C), R12.2, R24.2, U2.B7 (VSS), U2.EP (VSS), U2.F23 (VSS_PA), U3.16 (VSS), U3.32 (VSS), U3.33 (VSS)
- net I2C_SCL: now also R?.2, U3.13 (PA7)
- net I2C_SDA: now also R?.2, U3.27 (PB4); no longer R9.2
- net USB_DN: now also U2.AD4 (D-)
- net USB_DP: now also U2.AD6 (D+)
- net VBUS: now also U4.A3 (VIN), U4.A4 (VIN), U5.A3 (VIN), U5.A4 (VIN), R15.4; no longer D1.2 (A), Q1.5_6_7_8 (D), R6.1, TP1.1, USB1.A4 (VBUS), USB1.A9 (VBUS), USB1.B4 (VBUS), USB1.B9 (VBUS)
- net vSINK: now also U6.4 (VIN_SNS), U6.5 (VPWR), R15.1
- net at U5.A2 (RUN): now also U6.40 (VOUT_EN1), C13.2
- net at U5.D1 (FB): now also R20.1, R24.1
- net at U5.E1 (VOUT), U5.E2 (VOUT): now also R23.4
- net at U4.A2 (RUN): now also U6.41 (VOUT_EN0), C12.2
- net at U4.D1 (FB): now also R12.1, R17.1
- net at U4.E1 (VOUT), U4.E2 (VOUT): now also R13.4
- net at U6.1 (VIN_SNS_CAP): now also C6.1
- net at U6.10 (TSENSE0): now also C8.2, Q3.2 (E)
- net at U6.11 (TSENSE1): now also C9.2, Q4.2 (E)
- net at U6.14 (PG0): now also R16.2
- net at U6.15 (PG1): now also R21.2
- net at U6.17 (FAULTB0): now also R14.2
- net at U6.18 (FAULTB1): now also R22.2
- net I2C_SDA_SMBUS: now reaches U6.20 (SDA)
- net I2C_SDA_SMBUS: now also R?.2, U3.20 (PA10)
- net I2C_SCL_SMBUS: now reaches U6.21 (SCL)
- net I2C_SCL_SMBUS: now also R?.2, U3.19 (PA9)
- net at U6.23 (CONTROL0): now also R18.2
- net at U6.24 (CONTROL1): now also R19.2
- net at U6.28 (REFP): now also C7.2
- net at U6.29 (REFM): now also C7.1
- net at U6.30 (ISENSEP0): now also R13.3
- net at U6.31 (ISENSEM0): now also R13.2
- net at U6.32 (VSENSEP0): now also J1.1 (Pin_1), R13.1
- net at U6.34 (ISENSEP1): now also R23.3
- net at U6.35 (ISENSEM1): now also R23.2
- net at U6.36 (VSENSEP1): now also J2.1 (Pin_1), R23.1
- net at U6.38 (VDAC0): now also R17.2
- net at U6.39 (VDAC1): now also R20.2
- net at U6.43 (IIN_SNSP): now also R15.2
- net at U6.44 (IIN_SNSM): now also R15.3
- net at U6.6 (VDD33), U6.7 (VDD33): now also C11.2
- net at U6.8 (VDD25), U6.9 (VDD25): now also C10.2
- new net: D1.2 (A), Q1.5_6_7_8 (D), R6.1, TP1.1, USB1.A4 (VBUS), USB1.A9 (VBUS), USB1.B4 (VBUS), USB1.B9 (VBUS)
- new net: DBG1.4 (SWDCLK/TCK), U2.AA24 (SWDCLK)
- new net: DBG1.10 (~RESET~), U2.AC13 (P0.18/~RESET)
- new net: DBG1.2 (SWDIO/TMS), U2.AC24 (SWDIO)
- new net: R9.2, U3.4 (NRST)
- new net NRF_SWO: DBG1.6 (SWO/TDO), U2.AD22 (TRACEDATA0/P1.00)
- new net SMBUS_ALERT: U3.7 (PA1)
- new net SPI_MISO: U2.AC9 (P0.14), U3.12 (PA6)
- new net SPI_MOSI: U2.AD10 (P0.15), U3.22 (PA12)
- new net SPI_SCK: U2.AD8 (P0.13), U3.11 (PA5)
- new net SPI_SS: U2.AC11 (P0.16), U3.28 (PB5)
- new net STM32_SWDCLK: U3.24 (PA14)
- new net STM32_SWDIO: U3.23 (PA13)
- new net UART_RX: U2.AD12 (P0.17), U3.30 (PB7)
- new net UART_TX: U2.AC15 (P0.19), U3.29 (PB6)
- no-connect marks 11 -> 7
Other:
- note added: "for USB CDC\n"
- note removed: "Might switch to NRF52 due to PMBus compatibility issues \n"
- note removed: "add test header"
- moved on the sheet: C1, C2, C3, C4, C5, D1, JP1, JP2, Q1, Q2, R1, R11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

Commit message: integrated STM32 and assigned most footprints
Parts:
- removed R13, R23: R_Shunt_US, symbol Device:R_Shunt_US
- added C16: 1uF, Capacitor_SMD:C_0603_1608Metric, symbol Device:C
- added C18: 10uF, Capacitor_SMD:C_0603_1608Metric, symbol Device:C
- added D2: GREEN 0805, LED_SMD:LED_0805_2012Metric, symbol Device:LED
- added D3: RED 0805, LED_SMD:LED_0805_2012Metric, symbol Device:LED
- added R14, R15: 300, Resistor_SMD:R_0603_1608Metric, symbol Device:R_US
- added R18, R28: 20m, Resistor_SMD:R_1206_3216Metric, symbol Device:R_US
- added R30: 23.7k, Resistor_SMD:R_0603_1608Metric, symbol Device:R_US
- added R31: 76.8k, Resistor_SMD:R_0603_1608Metric, symbol Device:R_US
- added U7: LTM8074IY#PBF, LTM8074IY_PBF:BGA25C65P5X5_400X400X198N, symbol LTM8074IY_PBF:LTM8074IY#PBF
- C1: renamed from C2; footprint (none) -> Capacitor_SMD:C_0603_1608Metric
- C10: renamed from C6; footprint (none) -> Capacitor_SMD:C_0603_1608Metric
- C11: renamed from C7; footprint (none) -> Capacitor_SMD:C_0603_1608Metric
- C12: renamed from C8; footprint (none) -> Capacitor_SMD:C_0603_1608Metric
- C13: renamed from C9; footprint (none) -> Capacitor_SMD:C_0603_1608Metric
- C14: renamed from C10; value C -> .1uF; footprint (none) -> Capacitor_SMD:C_0603_1608Metric
- C15: renamed from C11; value C -> .1uF; footprint (none) -> Capacitor_SMD:C_0603_1608Metric
- C17: renamed from C13; footprint (none) -> Capacitor_SMD:C_0603_1608Metric
- C2, C3, C5: renamed from C?; footprint (none) -> Capacitor_SMD:C_0603_1608Metric
- C4: renamed from C3; footprint (none) -> Capacitor_SMD:C_0603_1608Metric
- C6: renamed from C12; footprint (none) -> Capacitor_SMD:C_0603_1608Metric
- C7: renamed from C4; footprint (none) -> Capacitor_SMD:C_0603_1608Metric
- C8: renamed from C5; footprint (none) -> Capacitor_SMD:C_0603_1608Metric
- C9: renamed from C1; footprint (none) -> Capacitor_SMD:C_0603_1608Metric
- D1: footprint (none) -> Diode_SMD:D_1206_3216Metric_Castellated
- JP1, JP2: footprint (none) -> Jumper:SolderJumper-2_P1.3mm_Bridged_RoundedPad1.0x1.5mm
- Q1, Q2: footprint TRANS_STL6P3LLH6 -> STL6P3LLH6:TRANS_STL6P3LLH6
- R1: renamed from R11; footprint (none) -> Resistor_SMD:R_0603_1608Metric
- R10, R11, R12, R6: renamed from R?; footprint (none) -> Resistor_SMD:R_0603_1608Metric
- R13: renamed from R3; footprint (none) -> Resistor_SMD:R_0603_1608Metric
- R16: renamed from R4; footprint (none) -> Resistor_SMD:R_0603_1608Metric
- R17: renamed from R12; footprint (none) -> Resistor_SMD:R_0603_1608Metric
- R19: renamed from R14; footprint (none) -> Resistor_SMD:R_0603_1608Metric
- R2: renamed from R6; footprint (none) -> Resistor_SMD:R_0603_1608Metric
- R20: renamed from R15; footprint (none) -> Resistor_SMD:R_0603_1608Metric
- R21: renamed from R16; footprint (none) -> Resistor_SMD:R_0603_1608Metric
- R22: renamed from R17; footprint (none) -> Resistor_SMD:R_0603_1608Metric
- R23: renamed from R18; footprint (none) -> Resistor_SMD:R_0603_1608Metric
- R24: renamed from R19; footprint (none) -> Resistor_SMD:R_0603_1608Metric
- R25: renamed from R20; footprint (none) -> Resistor_SMD:R_0603_1608Metric
- R26: renamed from R21; footprint (none) -> Resistor_SMD:R_0603_1608Metric
- R27: renamed from R22; footprint (none) -> Resistor_SMD:R_0603_1608Metric
- R29: renamed from R24; footprint (none) -> Resistor_SMD:R_0603_1608Metric
- R3: renamed from R7; footprint (none) -> Resistor_SMD:R_0603_1608Metric
- R4: renamed from R8; footprint (none) -> Resistor_SMD:R_0603_1608Metric
- R5: footprint (none) -> Resistor_SMD:R_0603_1608Metric
- R7: renamed from R9; footprint (none) -> Resistor_SMD:R_0603_1608Metric
- R8: renamed from R1; footprint Resistor_SMD:R_0805_2012Metric_Pad1.15x1.40mm_HandSolder -> Resistor_SMD:R_0603_1608Metric
- R9: renamed from R2; footprint (none) -> Resistor_SMD:R_0603_1608Metric
- TP1, TP2: footprint (none) -> TestPoint:TestPoint_Pad_D1.0mm
- U2: renamed from U1; footprint QFN50P400X400X90-25N -> STUSB4500QTR:QFN50P400X400X90-25N
- U4: footprint BGA25C65P5X5_400X400X198N -> LTM8074IY_PBF:BGA25C65P5X5_400X400X198N
- U6: renamed from U5; footprint BGA25C65P5X5_400X400X198N -> LTM8074IY_PBF:BGA25C65P5X5_400X400X198N
- USB1: footprint GCT_USB4085-GF-A_REVA -> USB4085-GF-A_REVA:GCT_USB4085-GF-A_REVA
- renumbered U2 to U1, U6 to U5
Connections:
- net +3V3: now also C18.1, U7.E1 (VOUT), U7.E2 (VOUT)
- net GND: now also U4.D5 (SYNC), U6.D5 (SYNC), C16.2, C18.2, R14.1, R15.1, R30.1, R31.1, U7.A1 (GND), U7.A5 (GND), U7.B2 (GND), U7.B3 (GND), U7.B4 (GND), U7.C2 (GND), U7.C3 (GND), U7.C4 (GND), U7.C5 (GND), U7.D2 (GND), U7.D3 (GND), U7.D4 (GND), U7.D5 (SYNC), U7.E3 (GND), U7.E4 (GND), U7.E5 (GND)
- net VUSB_RAW: now reaches D1.2 (A), Q1.5_6_7_8 (D), R2.1, TP1.1, USB1.A4 (VBUS), USB1.A9 (VBUS), USB1.B4 (VBUS), USB1.B9 (VBUS)
- net VUSB_RAW: now also C16.1, U7.A2 (RUN), U7.A3 (VIN), U7.A4 (VIN)
- net at U6.E1 (VOUT), U6.E2 (VOUT): now also U5.34 (ISENSEP1), R28.1
- net FAULTB0: now reaches R19.2, U5.17 (FAULTB0)
- net FAULTB0: now also U3.10 (PA4)
- net FAULTB1: now reaches R27.2, U5.18 (FAULTB1)
- net FAULTB1: now also U3.21 (PA11)
- net CONTROL0: now reaches R23.2, U5.23 (CONTROL0)
- net CONTROL0: now also U3.8 (PA2)
- net CONTROL1: now reaches R24.2, U5.24 (CONTROL1)
- net CONTROL1: now also U3.9 (PA3)
- net at U5.30 (ISENSEP0): now also U4.E1 (VOUT), U4.E2 (VOUT), R18.1
- net at U5.31 (ISENSEM0): now also J1.1 (Pin_1), U5.32 (VSENSEP0), R18.2
- net at U5.35 (ISENSEM1): now also J2.1 (Pin_1), U5.36 (VSENSEP1), R28.2
- net at U3.25 (PA15): now also D3.2 (A)
- net at U3.6 (PA0): now also D2.2 (A)
- new net: R30.2, U7.B5 (RT)
- new net: R31.2, U7.D1 (FB)
- new net: D3.1 (K), R15.2
- new net: D2.1 (K), R14.2
Other:
- note added: "1206"
- note added: "All resistors are 0603/1% unless specified\nAll caps are 0603 / 50v unless specified"
- moved on the sheet: C10, C14, C15, C2, C3, C5, R7

Commit message: added debug and power out connectors
Parts:
- removed DBG1: Cortex Debug, symbol Connector:Conn_ARM_JTAG_SWD_10
- removed R20: R_Shunt_US, Resistor_SMD:R_0603_1608Metric, symbol Device:R_Shunt_US
- added J3, J4: Connector, Connector_PinHeader_2.54mm:PinHeader_1x02_P2.54mm_Vertical, symbol Connector:Conn_01x02_Male
- added PH1, PH2: FTSH-105-01-L-DV-K, SAMTEC_FTSH-105-01-L-DV-K, symbol FTSH-105-01-L-DV-K:FTSH-105-01-L-DV-K
- added R20: 20m, Resistor_SMD:R_1206_3216Metric, symbol Device:R_US
- added R32, R33: 40.2k, Resistor_SMD:R_0603_1608Metric, symbol Device:R_US
- added R34: 10k, Resistor_SMD:R_0603_1608Metric, symbol Device:R_US
- added TP3, TP4: TestPoint, TestPoint:TestPoint_Pad_D1.0mm, symbol Connector:TestPoint
- J1, J2: footprint (none) -> Connector_AMASS:AMASS_XT30PW-F_1x02_P2.50mm_Horizontal
Connections:
- net +3V3: now also PH1.1 (VTref), PH2.1 (VTref), R34.1
- net GND: now also J1.1 (Pin_1), J2.1 (Pin_1), J3.1 (Pin_1), J4.1 (Pin_1), PH1.3 (GND), PH1.5 (GND), PH1.9 (GDET), PH2.3 (GND), PH2.5 (GND), PH2.9 (GDET), R32.2, R33.2; no longer J1.2 (Pin_2), J2.2 (Pin_2)
- net NRF_SWO: now also PH2.6 (SWO)
- net STM32_SWDCLK: now also PH1.4 (SWDCLK)
- net STM32_SWDIO: now also PH1.2 (SWDIO)
- net STUSB_ALERT: now also U3.18 (PA8)
- net VBUS: now also U5.44 (IIN_SNSM), R20.2
- net vSINK: now also U5.43 (IIN_SNSP), R20.1
- net at U6.B5 (RT): now also R33.1
- net at R18.2, U5.31 (ISENSEM0), U5.32 (VSENSEP0): now also J1.2 (Pin_2), J3.2 (Pin_2); no longer J1.1 (Pin_1)
- net at R28.2, U5.35 (ISENSEM1), U5.36 (VSENSEP1): now also J2.2 (Pin_2), J4.2 (Pin_2); no longer J2.1 (Pin_1)
- net at U4.B5 (RT): now also R32.1
- net NRF_SWDCLK: now reaches U1.AA24 (SWDCLK)
- net NRF_SWDCLK: now also PH2.4 (SWDCLK)
- net NRF_NRST: now reaches U1.AC13 (P0.18/~RESET)
- net NRF_NRST: now also PH2.10 (nRST), R34.2
- net NRF_SWDIO: now reaches U1.AC24 (SWDIO)
- net NRF_SWDIO: now also PH2.2 (SWDIO)
- net at U3.2 (PC14): now also TP3.1
- net STM32_SWO: now reaches U3.26 (PB3)
- net STM32_SWO: now also PH1.6 (SWO)
- net at U3.3 (PC15): now also TP4.1
- net STM32_NRST: now reaches R7.2, U3.4 (NRST)
- net STM32_NRST: now also PH1.10 (nRST)
Other:
- moved on the sheet: C2, C3, C5, D2, D3, J1, J2, R10, R11, R12, R14, R15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
